File: Electronics/flag-badge/_restore_backup_2026-08-28T23-02-19-014/flag-badge.kicad_sch (KiCad schematic)
At the start: 43 parts, among them J1 USB_C_Receptacle_USB2.0_14P, J2 Conn_01x01_Pin, J3 Conn_01x01_Pin, J4 Conn_01x03_Pin, J8 Conn_01x12_Pin, SW1 SW_Push, U1 BQ24075RGT, U2 W25Q128JVS, U3 XC6220B331MR, U4 RP2040, Y1 Crystal_GND24

Commit message: PCB
Parts:
- removed R10: 1k5, Resistor_SMD:R_0201_0603Metric, symbol k:R
- removed R11: 1k, Resistor_SMD:R_0201_0603Metric, symbol k:R
- added D2, D3: 1N5817, Diode_THT:D_DO-41_SOD81_P10.16mm_Horizontal, symbol k:1N5817
- J1: footprint Connector_USB:USB_C_Receptacle_HRO_TYPE-C-31-M-12 -> Connector_USB:USB_C_Receptacle_Molex_105450-0101
- J8: footprint Connector_FFC-FPC:Molex_200528-0120_1x12-1MP_P1.00mm_Horizontal -> Connector_FFC-FPC:TE_1-84952-8_1x18-1MP_P1.0mm_Horizontal
- SW1: footprint Button_Switch_SMD:SW_Push_SPST_NO_Alps_SKRK -> Button_Switch_SMD:SW_DIP_SPSTx01_Slide_6.7x4.1mm_W6.73mm_P2.54mm_LowProfile_JPin
Connections:
- net +5V: now also C19.1, U1.13 (IN), D2.1 (K), D3.1 (K); no longer C1.1, C18.1, R8.2, R9.2, U1.10 (OUT), U1.11 (OUT), U1.5 (EN2), U3.1 (VIN), U3.3 (CE)
- net GND: no longer J1.SH (SHIELD), U1.17 (VSS), U1.8 (VSS)
- net USB_5V: now also D2.2 (A); no longer C19.1, U1.13 (IN)
- net SYSOFF: no longer names the net of U1.15 (SYSOFF)
- net SYSOFF: no longer U4.38 (GPIO26/ADC0)
- new net: U1.17 (VSS), U1.8 (VSS)
- new net +5V_BAT: C1.1, U3.1 (VIN), U3.3 (CE)
- new net BAT_O: C18.1, D3.2 (A), R8.2, R9.2, U1.10 (OUT), U1.11 (OUT), U1.5 (EN2)
Other:
- moved on the sheet: J1, R1, R2, R3, R4
